File: kicad/Whiplaesh.kicad_sch (KiCad schematic)
At the start: 82 parts, among them SW1 SW_PUSH, SW10 SW_PUSH, SW11 SW_PUSH, SW12 SW_PUSH, SW13 SW_PUSH, SW14 SW_PUSH, SW15 SW_PUSH, SW16 SW_PUSH, SW17 SW_PUSH, SW18 SW_PUSH, SW19 SW_PUSH, SW2 SW_PUSH, SW20 SW_PUSH, SW21 SW_PUSH, SW22 SW_PUSH, SW23 SW_PUSH, SW24 SW_PUSH, SW25 SW_PUSH, SW26 SW_PUSH, SW27 SW_PUSH, SW28 SW_PUSH, SW29 SW_PUSH, SW3 SW_PUSH, SW30 SW_PUSH, SW31 SW_PUSH, SW32 SW_PUSH, SW4 SW_PUSH, SW5 SW_PUSH, SW6 SW_PUSH, SW7 SW_PUSH, SW8 SW_PUSH, SW9 SW_PUSH

Commit message: Redo routing, add ground plane, add fingerpunch footprints
Parts:
- MCU1, MCU2: footprint footprints:MCU_nice-nano -> library:ArduinoProMicro
- VIK_OUT1, VIK_OUT2: value ~ -> (none)
Changed lines of the file:
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@@
 			)
 		)
-		(property "Footprint" "footprints:MCU_nice-nano"
+		(property "Footprint" "library:ArduinoProMicro"
 			(at 77.47 257.81 90)
 			(effects
@@
 			)
 		)
-		(property "Value" "~"
+		(property "Value" ""
 			(at 121.92 205.74 0)
 			(effects
@@
 			)
 		)
-		(property "Footprint" "footprints:MCU_nice-nano"
+		(property "Footprint" "library:ArduinoProMicro"
 			(at 77.47 118.11 90)
 			(effects
@@
 			)
 		)
-		(property "Value" "~"
+		(property "Value" ""
 			(at 121.92 66.04 0)
 			(effects
