File: kicad/Whiplaesh.kicad_pcb (KiCad board)
At the start: 2 copper layers, 126.1 x 106.1 mm, 42 parts

Commit message: add right board in ergogen config
Connections:
- D1 pad 1: P6 -> (no net)
- D10 pad 1: P5 -> (no net)
- D11 pad 1: P4 -> (no net)
- D12 pad 1: P6 -> (no net)
- D13 pad 1: P5 -> (no net)
- D14 pad 1: P4 -> (no net)
- D15 pad 1: P8 -> (no net)
- D16 pad 1: P8 -> (no net)
- D2 pad 1: P5 -> (no net)
- D3 pad 1: P6 -> (no net)
- D4 pad 1: P5 -> (no net)
- D5 pad 1: P4 -> (no net)
- D6 pad 1: P6 -> (no net)
- D7 pad 1: P5 -> (no net)
- D8 pad 1: P4 -> (no net)
- D9 pad 1: P6 -> (no net)
- SW1 pad 1: P19 -> (no net)
- SW10 pad 1: P14 -> (no net)
- SW11 pad 1: P14 -> (no net)
- SW12 pad 1: P16 -> (no net)
- SW13 pad 1: P16 -> (no net)
- SW14 pad 1: P16 -> (no net)
- SW15 pad 1: P14 -> (no net)
- SW16 pad 1: P16 -> (no net)
- SW2 pad 1: P19 -> (no net)
- SW3 pad 1: P18 -> (no net)
- SW4 pad 1: P18 -> (no net)
- SW5 pad 1: P18 -> (no net)
- SW6 pad 1: P15 -> (no net)
- SW7 pad 1: P15 -> (no net)
- SW8 pad 1: P15 -> (no net)
- SW9 pad 1: P14 -> (no net)

Commit message: Remove nice!view and update schematics and pcb
Parts:
- removed DISP1: , ceoloide:display_nice_view
- added D17: 1N4148W, fingerpunch:D3_TH_SMD, B.Cu at (243.0, 83.6)
- added D18: 1N4148W, fingerpunch:D3_TH_SMD, B.Cu at (263.8, 94.8)
- added D19: 1N4148W, fingerpunch:D3_TH_SMD, B.Cu at (39.7, 113.5)
- added D20: 1N4148W, fingerpunch:D3_TH_SMD, B.Cu at (57.2, 102.5)
- added D21: 1N4148W, fingerpunch:D3_TH_SMD, B.Cu at (76.2, 93.0)
- added D22: 1N4148W, fingerpunch:D3_TH_SMD, B.Cu at (95.2, 97.8)
- added D23: 1N4148W, fingerpunch:D3_TH_SMD, B.Cu at (114.2, 102.5)
- added D24: 1N4148W, fingerpunch:D3_TH_SMD, B.Cu at (186.0, 102.6)
- added D25: 1N4148W, fingerpunch:D3_TH_SMD, B.Cu at (205.0, 97.8)
- added D26: 1N4148W, fingerpunch:D3_TH_SMD, B.Cu at (224.0, 93.1)
- added D27: 1N4148W, fingerpunch:D3_TH_SMD, B.Cu at (243.0, 102.6)
- added D28: 1N4148W, fingerpunch:D3_TH_SMD, B.Cu at (260.5, 113.5)
- added D29: 1N4148W, fingerpunch:D3_TH_SMD, B.Cu at (106.6, 129.4)
- added D30: 1N4148W, fingerpunch:D3_TH_SMD, B.Cu at (124.9, 134.3)
- added D31: 1N4148W, fingerpunch:D3_TH_SMD, B.Cu at (175.3, 134.4)
- added D32: 1N4148W, fingerpunch:D3_TH_SMD, B.Cu at (193.6, 129.4)
- added G***: LOGO, library:Aespa, F.Cu at (73.7, 79.4)
- added G***: LOGO, library:Aespa, F.Cu at (211.1, 79.7)
- added H5: MountingHole, MountingHole:MountingHole_2.2mm_M2, F.Cu at (256.3, 54.6)
- added H6: MountingHole, MountingHole:MountingHole_2.2mm_M2, F.Cu at (190.7, 43.2)
- added H7: MountingHole, MountingHole:MountingHole_2.2mm_M2, F.Cu at (205.2, 121.1)
- added H8: MountingHole, MountingHole:MountingHole_2.2mm_M2, F.Cu at (247.7, 116.3)
- added JST2: JST_PH, Connector_JST:JST_PH_S2B-PH-K_1x02_P2.00mm_Horizontal, B.Cu at (164.9, 81.3)
- added MCU2: ~, footprints:MCU_nice-nano, F.Cu at (165.1, 59.6)
- added PWR2: OS102011MA1QN1, footprints:OS102011MA1QN1_CNK, F.Cu at (156.6, 123.3)
- added RST2: SW_PUSH, footprints:SW_SKHLACA010_ALPS, F.Cu at (154.6, 80.1)
- added SW17: SW_PUSH, fingerpunch:gateron-ks27-choc-v1-mx-soldered-and-hotswap, F.Cu at (243.0, 73.6)
- added SW18: SW_PUSH, fingerpunch:gateron-ks27-choc-v1-mx-soldered-and-hotswap, F.Cu at (265.5, 85.0)
- added SW19: SW_PUSH, fingerpunch:gateron-ks27-choc-v1-mx-soldered-and-hotswap, F.Cu at (38.0, 103.7)
- added SW20: SW_PUSH, fingerpunch:gateron-ks27-choc-v1-mx-soldered-and-hotswap, F.Cu at (57.2, 92.5)
- added SW21: SW_PUSH, fingerpunch:gateron-ks27-choc-v1-mx-soldered-and-hotswap, F.Cu at (76.2, 83.0)
- added SW22: SW_PUSH, fingerpunch:gateron-ks27-choc-v1-mx-soldered-and-hotswap, F.Cu at (95.2, 87.8)
- added SW23: SW_PUSH, fingerpunch:gateron-ks27-choc-v1-mx-soldered-and-hotswap, F.Cu at (114.2, 92.5)
- added SW24: SW_PUSH, fingerpunch:gateron-ks27-choc-v1-mx-soldered-and-hotswap, F.Cu at (186.0, 92.6)
- added SW25: SW_PUSH, fingerpunch:gateron-ks27-choc-v1-mx-soldered-and-hotswap, F.Cu at (205.0, 87.8)
- added SW26: SW_PUSH, fingerpunch:gateron-ks27-choc-v1-mx-soldered-and-hotswap, F.Cu at (224.0, 83.1)
- added SW27: SW_PUSH, fingerpunch:gateron-ks27-choc-v1-mx-soldered-and-hotswap, F.Cu at (243.0, 92.6)
- added SW28: SW_PUSH, fingerpunch:gateron-ks27-choc-v1-mx-soldered-and-hotswap, F.Cu at (262.2, 103.7)
- added SW29: SW_PUSH, fingerpunch:gateron-ks27-choc-v1-mx-soldered-and-hotswap, F.Cu at (109.2, 119.8)
- added SW30: SW_PUSH, fingerpunch:gateron-ks27-choc-v1-mx-soldered-and-hotswap, F.Cu at (127.5, 124.7)
- added SW31: SW_PUSH, fingerpunch:gateron-ks27-choc-v1-mx-soldered-and-hotswap, F.Cu at (172.7, 124.7)
- added SW32: SW_PUSH, fingerpunch:gateron-ks27-choc-v1-mx-soldered-and-hotswap, F.Cu at (191.1, 119.8)
- added VIK_OUT2: ~, vik:vik-keyboard-connector-horizontal, F.Cu at (165.1, 102.0)
- added mouse-bite-5mm-slot: VAL**, library:mouse-bite-5mm-slot, F.Cu at (150.1, 62.9)
- added mouse-bite-5mm-slot: VAL**, library:mouse-bite-5mm-slot, F.Cu at (150.1, 107.8)
- D1, D10, D11, D12, D13, D14, D15, D16, D2, D3, D4, D5, D6, D7, D8, D9: value (none) -> 1N4148W; footprint ceoloide:diode_tht_sod123 -> fingerpunch:D3_TH_SMD
- H1, H2, H3, H4: value (none) -> MountingHole; footprint ceoloide:mounting_hole_plated -> MountingHole:MountingHole_2.2mm_M2
- JST1: value (none) -> JST_PH; footprint ceoloide:battery_connector_jst_ph_2 -> Connector_JST:JST_PH_S2B-PH-K_1x02_P2.00mm_Horizontal
- MCU1: value (none) -> ~; footprint ceoloide:mcu_nice_nano -> footprints:MCU_nice-nano
- PWR1: value (none) -> OS102011MA1QN1; footprint ceoloide:power_switch_smd_side -> footprints:OS102011MA1QN1_CNK
- RST1: value (none) -> SW_PUSH; footprint ceoloide:reset_switch_tht_top -> footprints:SW_SKHLACA010_ALPS
- SW1, SW10, SW11, SW12, SW13, SW14, SW15, SW16, SW2, SW3, SW4, SW5, SW6, SW7, SW8, SW9: value (none) -> SW_PUSH; footprint ks27-choc-v1-mx-soldered-and-hotswap -> fingerpunch:gateron-ks27-choc-v1-mx-soldered-and-hotswap; moved to F.Cu
- VIK_OUT1: value vik-keyboard-connector-horizontal -> ~; footprint vik-keyboard-connector-horizontal -> vik:vik-keyboard-connector-horizontal
- moved D8 113.9 mm to (243.0, 64.6)
- moved SW8 113.9 mm to (243.0, 54.6)
- moved SW9 113.7 mm to (34.7, 84.9), turned to 10 degrees
- moved D9 112.0 mm to (36.4, 94.8), turned to 10 degrees
- moved D7 97.7 mm to (224.0, 55.1)
- moved SW7 97.7 mm to (224.0, 45.1)
- moved D10 90.9 mm to (57.2, 83.5)
- moved SW10 90.9 mm to (57.2, 73.5)
- moved D6 84.7 mm to (205.0, 59.8)
- moved SW6 84.7 mm to (205.0, 49.8)
- moved D16 79.6 mm to (224.0, 74.1), turned to 0 degrees
- moved SW16 78.5 mm to (224.0, 64.1), turned to 0 degrees
- moved D12 77.3 mm to (95.2, 78.8)
- moved SW12 77.3 mm to (95.2, 68.8)
- moved D5 75.9 mm to (186.0, 64.6)
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Connections:
- net P0 renamed RGB
- net P1 renamed CS
- net P10 renamed MOSI
- net P2 renamed SDA
- net P3 renamed SCL
- net P4 renamed MISO
- net P9 renamed SCLK
- D1 pad 1: (no net) -> ROW0
- D1 pad 2: pinky_bottom -> Net-(D1-A)
- D10 pad 1: (no net) -> ROW1
- D10 pad 2: index_home -> Net-(D10-A)
- D11 pad 1: (no net) -> ROW1
- D11 pad 2: index_top -> Net-(D11-A)
- D12 pad 1: (no net) -> ROW1
- D12 pad 2: inner_bottom -> Net-(D12-A)
- D13 pad 1: (no net) -> ROW1
- D13 pad 2: inner_home -> Net-(D13-A)
- D14 pad 1: (no net) -> ROW1_r
- D14 pad 2: inner_top -> Net-(D14-A)
- D15 pad 1: (no net) -> ROW1_r
- D15 pad 2: left_cluster -> Net-(D15-A)
- D16 pad 1: (no net) -> ROW1_r
- D16 pad 2: right_cluster -> Net-(D16-A)
- D2 pad 1: (no net) -> ROW0
- D2 pad 2: pinky_home -> Net-(D2-A)
- D3 pad 1: (no net) -> ROW0
- D3 pad 2: ring_bottom -> Net-(D3-A)
- D4 pad 1: (no net) -> ROW0
- D4 pad 2: ring_home -> Net-(D4-A)
- D5 pad 1: (no net) -> ROW0_r
- D5 pad 2: ring_top -> Net-(D5-A)
- D6 pad 1: (no net) -> ROW0_r
- D6 pad 2: middle_bottom -> Net-(D6-A)
- D7 pad 1: (no net) -> ROW0_r
- D7 pad 2: middle_home -> Net-(D7-A)
- D8 pad 1: (no net) -> ROW0_r
- D8 pad 2: middle_top -> Net-(D8-A)
- D9 pad 1: (no net) -> ROW1
- D9 pad 2: index_bottom -> Net-(D9-A)
- MCU1 pad 10: P7 -> ROW2
- MCU1 pad 11: P8 -> ROW3
- MCU1 pad 14: P16 -> COL4
- MCU1 pad 15: P14 -> COL3
- MCU1 pad 16: P15 -> COL2
- MCU1 pad 17: P18 -> COL1
- MCU1 pad 18: P19 -> COL0
- MCU1 pad 19: P20 -> GPIO_AD1
- MCU1 pad 20: P21 -> GPIO_AD2
- MCU1 pad 24: RAW -> +5V
- MCU1 pad 8: P5 -> ROW0
- MCU1 pad 9: P6 -> ROW1
- PWR1 pad 1: (no net) -> +5V
- PWR1 pad 2: RAW -> BAT_P
- PWR1 pad 3: BAT_P -> unconnected-(PWR1-Pad3)
- RST1 pad 1: RST -> GND
- RST1 pad 2: GND -> RST
- SW1 pad 1: (no net) -> Net-(D1-A)
- SW1 pad 2: pinky_bottom -> COL1
- SW10 pad 1: (no net) -> Net-(D10-A)
- SW10 pad 2: index_home -> COL1
- SW11 pad 1: (no net) -> Net-(D11-A)
- SW11 pad 2: index_top -> COL2
- SW12 pad 1: (no net) -> Net-(D12-A)
- SW12 pad 2: inner_bottom -> COL3
- SW13 pad 1: (no net) -> Net-(D13-A)
- SW13 pad 2: inner_home -> COL4
- SW14 pad 1: (no net) -> Net-(D14-A)
- SW14 pad 2: inner_top -> COL0_r
- SW15 pad 1: (no net) -> Net-(D15-A)
- SW15 pad 2: left_cluster -> COL1_r
- SW16 pad 1: (no net) -> Net-(D16-A)
- SW16 pad 2: right_cluster -> COL2_r
- SW2 pad 1: (no net) -> Net-(D2-A)
- SW2 pad 2: pinky_home -> COL2
- SW3 pad 1: (no net) -> Net-(D3-A)
- SW3 pad 2: ring_bottom -> COL3
- SW4 pad 1: (no net) -> Net-(D4-A)
- SW4 pad 2: ring_home -> COL4
- SW5 pad 1: (no net) -> Net-(D5-A)
- SW5 pad 2: ring_top -> COL1_r
- SW6 pad 1: (no net) -> Net-(D6-A)
- SW6 pad 2: middle_bottom -> COL2_r
- SW7 pad 1: (no net) -> Net-(D7-A)
- SW7 pad 2: middle_home -> COL3_r
- SW8 pad 1: (no net) -> Net-(D8-A)
- SW8 pad 2: middle_top -> COL4_r
- SW9 pad 1: (no net) -> Net-(D9-A)
- SW9 pad 2: index_bottom -> COL0
- VIK_OUT1 pad 6: RAW -> +5V
- VIK_OUT1 pad 7: P21 -> GPIO_AD1
- VIK_OUT1 pad 9: P20 -> GPIO_AD2
Routing:
- net (no net): track 419.4 -> 0.00 mm
- net COL4_r: track 0.00 -> 312.3 mm, vias 0 -> 1
- net COL3_r: track 0.00 -> 308.4 mm, vias 0 -> 3
- net COL3: track 0.00 -> 223.9 mm
- net COL0: track 0.00 -> 220.9 mm
- net COL1: track 0.00 -> 207.4 mm
- net COL4: track 0.00 -> 206.3 mm
- net COL2: track 0.00 -> 185.6 mm
- net COL2_r: track 0.00 -> 162.7 mm, vias 0 -> 1
- net ROW2: track 0.00 -> 145.2 mm
- net ROW2_r: track 0.00 -> 144.2 mm
- net COL1_r: track 0.00 -> 139.8 mm, vias 0 -> 1
- net ROW1_r: track 0.00 -> 133.7 mm, vias 0 -> 4
- net ROW1: track 0.00 -> 130.4 mm
- net ROW0_r: track 0.00 -> 101.4 mm, vias 0 -> 3
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Other:
- board size 126.1 x 106.1 mm -> 257.1 x 106.2 mm
- board text added: "JLCJLCJLCJLC"
- board text added: "by ykz89"

Commit message: Redo routing, add ground plane, add fingerpunch footprints
Parts:
- added REF**: vik-logo-small, vik:vik-logo-small, F.Cu at (133.6, 71.9)
- added REF**: vik-logo-small, vik:vik-logo-small, F.Cu at (164.7, 71.3)
- D1, D10, D11, D12, D13, D14, D15, D16, D17, D18, D19, D2, D20, D21, D22, D23, D24, D25, D26, D27, D28, D29, D3, D30, D31, D32, D4, D5, D6, D7, D8, D9: footprint fingerpunch:D3_TH_SMD -> Diode_SMD:D_SOD-123
- MCU1, MCU2: footprint footprints:MCU_nice-nano -> library:ArduinoProMicro
- moved H7 45.2 mm to (162.4, 135.8)
- moved H3 45.2 mm to (137.8, 135.8)
- moved D19 17.4 mm to (30.0, 99.0)
- moved D9 17.4 mm to (26.7, 80.3)
- moved D31 17.2 mm to (164.6, 120.8)
- moved D32 17.2 mm to (183.0, 115.9)
- moved D29 17.2 mm to (104.2, 112.4)
- moved D30 17.2 mm to (122.5, 117.3)
- moved D15 17.2 mm to (198.2, 63.0)
- moved D16 17.2 mm to (217.2, 58.3)
- moved D5 17.2 mm to (179.2, 48.8)
- moved D7 17.2 mm to (217.2, 39.3)
- moved D8 17.2 mm to (236.2, 48.8)
- moved D14 17.2 mm to (179.2, 67.8)
- moved D17 17.2 mm to (236.2, 67.8)
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Routing:
- net COL4_r: track 312.3 -> 368.4 mm, vias 1 -> 3
- net GND: track 88.7 -> 35.0 mm, vias 3 -> 2
- net COL3_r: track 308.4 -> 359.7 mm, vias 3 -> 5
- net COL2_r: track 162.7 -> 207.5 mm, vias 1 -> 4
- net COL1_r: track 139.8 -> 180.3 mm, vias 1 -> 4
- net VCC_r: track 58.0 -> 97.6 mm, vias 5 -> 2
- net SCLK: track 31.2 -> 68.8 mm, vias 0 -> 2
- net GPIO_AD2: track 50.6 -> 88.1 mm, vias 0 -> 2
- net MISO: track 44.1 -> 80.9 mm, vias 0 -> 2
- net SDA_r: track 55.9 -> 89.8 mm, vias 4 -> 2
- net MOSI: track 32.6 -> 65.9 mm, vias 0 -> 2
- net CS: track 61.7 -> 93.8 mm, vias 0 -> 2
- net GPIO_AD1: track 48.6 -> 77.7 mm, vias 1 -> 2
- net GPIO_AD1_r: track 47.8 -> 76.6 mm
- net COL1: track 207.4 -> 234.9 mm, vias 0 -> 4
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- added copper zone on B.Cu, net GND
- added copper zone on F.Cu, net GND
- added copper zone on B.Cu, net GND_r
- added copper zone on F.Cu, net GND_r

Commit message: Fix silkscreen, add production files
Parts:
- moved G*** 0.92 mm to (210.2, 79.7)
- moved G*** 0.38 mm to (74.0, 79.7)
Changed lines of the file:
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@@
 			(unlocked yes)
 			(layer "F.SilkS")
+			(hide yes)
 			(effects
 				(font
@@
 			(unlocked yes)
 			(layer "F.SilkS")
+			(hide yes)
 			(effects
 				(font
@@
 			(unlocked yes)
 			(layer "F.SilkS")
+			(hide yes)
 			(effects
 				(font
@@
 			(unlocked yes)
 			(layer "F.SilkS")
+			(hide yes)
 			(effects
 				(font
@@
 			(unlocked yes)
 			(layer "F.SilkS")
+			(hide yes)
 			(effects
 				(font
@@
 		(fp_arc
 			(start 2.464162 0.61604)
-			(mid 1.563148 2.002043)
+			(mid 1.563149 2.002043)
 			(end 0 2.54)
 			(stroke
@@
 		(fp_arc
 			(start 2.464162 0.61604)
-			(mid 1.563148 2.002043)
+			(mid 1.563149 2.002043)
 			(end 0 2.54)
 			(stroke
@@
 			(unlocked yes)
 			(layer "F.SilkS")
+			(hide yes)
 			(effects
 				(font
@@
 			(unlocked yes)
 			(layer "F.SilkS")
+			(hide yes)
 			(effects
 				(font
@@
 		(fp_arc
 			(start 6.35 4.445)
-			(mid 5.606052 6.241053)
+			(mid 5.606053 6.241053)
 			(end 3.81 6.985)
 			(stroke
@@
 		(fp_arc
 			(start 6.35 4.445)
-			(mid 5.606052 6.241053)
+			(mid 5.606053 6.241053)
 			(end 3.81 6.985)
 			(stroke
@@
 			(unlocked yes)
 			(layer "F.SilkS")
+			(hide yes)
 			(effects
 				(font
@@
 			(unlocked yes)
 			(layer "F.SilkS")
+			(hide yes)
 			(effects
 				(font
@@
 		)
 		(pad "2" smd rect
-			(at 5.875 5.750002 10)
+			(at 5.875 5.750003 10)
 			(size 2.6 2.6)
 			(layers "B.Cu" "B.Paste" "B.Mask")
@@
 			(at 0 -3.2 0)
 			(layer "F.SilkS")
+			(hide yes)
 			(effects
 				(font
@@
 			(unlocked yes)
 			(layer "F.SilkS")
+			(hide yes)
 			(effects
 				(font
@@
 			(unlocked yes)
 			(layer "F.SilkS")
+			(hide yes)
 			(effects
 				(font
@@
 			(unlocked yes)
 			(layer "F.SilkS")
+			(hide yes)
 			(effects
 				(font
@@
 			(unlocked yes)
 			(layer "F.SilkS")
+			(hide yes)
 			(effects
 				(font
@@
 			(unlocked yes)
 			(layer "F.SilkS")
+			(hide yes)
 			(effects
 				(font
@@
 			(unlocked yes)
 			(layer "F.SilkS")
+			(hide yes)
 			(effects
 				(font
@@
 			(unlocked yes)
 			(layer "F.SilkS")
+			(hide yes)
 			(effects
 				(font
@@
 	(footprint "library:Aespa"
 		(layer "F.Cu")
-		(at 73.7 79.4)
+		(at 73.954385 79.684966)
 		(property "Reference" "G***"
 			(at 0 0 0)
@@
 			(at 0 -3.2 0)
 			(layer "F.SilkS")
+			(hide yes)
 			(effects
 				(font
@@
 			(unlocked yes)
 			(layer "F.SilkS")
+			(hide yes)
 			(effects
 				(font
@@
 		)
 		(pad "2" smd rect
-			(at 5.875 5.750002 10)
+			(at 5.875 5.750003 10)
 			(size 2.6 2.6)
 			(layers "B.Cu" "B.Paste" "B.Mask")
@@
 			(unlocked yes)
 			(layer "F.SilkS")
+			(hide yes)
 			(effects
 				(font
@@
 			(at 0 -3.2 0)
 			(layer "F.SilkS")
+			(hide yes)
 			(effects
 				(font
@@
 			(unlocked yes)
 			(layer "F.SilkS")
+			(hide yes)
 			(effects
 				(font
@@
 			(unlocked yes)
 			(layer "F.SilkS")
+			(hide yes)
 			(effects
 				(font
@@
 	(footprint "library:Aespa"
 		(layer "F.Cu")
-		(at 211.1 79.7)
+		(at 210.184385 79.684966)
 		(property "Reference" "G***"
 			(at 0 0 0)
@@
 			(at 0 -3.2 0)
 			(layer "F.SilkS")
+			(hide yes)
 			(effects
 				(font
@@
 			(unlocked yes)
 			(layer "F.SilkS")
+			(hide yes)
 			(effects
 				(font
@@
 			(at 0 -3.2 0)
 			(layer "F.SilkS")
+			(hide yes)
 			(effects
 				(font
@@
 			(unlocked yes)
 			(layer "F.SilkS")
+			(hide yes)
 			(effects
 				(font
@@
 			(unlocked yes)
 			(layer "F.SilkS")
+			(hide yes)
 			(effects
 				(font
@@
 			(unlocked yes)
 			(layer "F.SilkS")
+			(hide yes)
 			(effects
 				(font
@@
 			(unlocked yes)
 			(layer "F.SilkS")
+			(hide yes)
 			(effects
 				(font
@@
 			(at 0 -3.2 0)
 			(layer "F.SilkS")
+			(hide yes)
 			(effects
 				(font
@@
 			(unlocked yes)
 			(layer "F.SilkS")
+			(hide yes)
 			(effects
 				(font
@@
 			(unlocked yes)
 			(layer "F.SilkS")
+			(hide yes)
 			(effects
 				(font
@@
 			(unlocked yes)
 			(layer "F.SilkS")
+			(hide yes)
 			(effects
 				(font
@@
 			(unlocked yes)
 			(layer "F.SilkS")
+			(hide yes)
 			(effects
 				(font
@@
 		(fp_arc
 			(start 2.464162 0.61604)
-			(mid 1.563148 2.002043)
+			(mid 1.563149 2.002043)
 			(end 0 2.54)
 			(stroke
@@
 		(fp_arc
 			(start 2.464162 0.61604)
-			(mid 1.563148 2.002043)
+			(mid 1.563149 2.002043)
 			(end 0 2.54)
 			(stroke
@@
 			(unlocked yes)
 			(layer "F.SilkS")
+			(hide yes)
 			(effects
 				(font
@@
 		(fp_arc
 			(start 6.35 4.445)
-			(mid 5.606052 6.241053)
+			(mid 5.606053 6.241053)
 			(end 3.81 6.985)
 			(stroke
@@
 		(fp_arc
 			(start 6.35 4.445)
-			(mid 5.606052 6.241053)
+			(mid 5.606053 6.241053)
 			(end 3.81 6.985)
 			(stroke
@@
 			(unlocked yes)
 			(layer "F.SilkS")
+			(hide yes)
 			(effects
 				(font
@@
 			(unlocked yes)
 			(layer "F.SilkS")
+			(hide yes)
 			(effects
 				(font
@@
 			(at 0 -3.2 0)
 			(layer "F.SilkS")
+			(hide yes)
 			(effects
 				(font
@@
 	)
 	(gr_text "Whiplaesh"
-		(at 133.4 57.7 90)
+		(at 133.33 58.16 90)
 		(layer "F.SilkS")
 		(effects
