File: kicad/Whiplaesh.kicad_pcb (KiCad board)
At the start: 2 copper layers, 257.1 x 106.2 mm, 88 parts, among them SW1 SW_PUSH, SW10 SW_PUSH, SW11 SW_PUSH, SW12 SW_PUSH, SW13 SW_PUSH, SW14 SW_PUSH, SW15 SW_PUSH, SW16 SW_PUSH, SW17 SW_PUSH, SW18 SW_PUSH, SW19 SW_PUSH, SW2 SW_PUSH, SW20 SW_PUSH, SW21 SW_PUSH, SW22 SW_PUSH, SW23 SW_PUSH, SW24 SW_PUSH, SW25 SW_PUSH, SW26 SW_PUSH, SW27 SW_PUSH, SW28 SW_PUSH, SW29 SW_PUSH, SW3 SW_PUSH, SW30 SW_PUSH, SW31 SW_PUSH, SW32 SW_PUSH, SW4 SW_PUSH, SW5 SW_PUSH, SW6 SW_PUSH, SW7 SW_PUSH, SW8 SW_PUSH, SW9 SW_PUSH

Commit message: Tentatively add bottom plate
Routing:
- net COL4_r: track 368.4 -> 384.4 mm
- net ROW3: track 67.9 -> 72.6 mm, vias 0 -> 1
- net COL3_r: track 359.7 -> 364.3 mm

Commit message: Mirror ground fill, fix battery connector position
Parts:
- moved JST2 2.06 mm to (165.1, 83.4)
Routing:
- net ROW3_r: track 87.3 -> 72.7 mm
- net BAT_P_r: track 53.8 -> 52.5 mm
- net GND_r: track 62.0 -> 60.8 mm
- net Net-(D22-A): track 21.1 -> 22.3 mm
- net Net-(D19-A): track 20.5 -> 21.6 mm
- net VCC_r: track 97.6 -> 98.1 mm
